Commit message: modif scripts

File: urdf/my_robot_arm.xacro (robot description, xacro)
@@ -3,5 +3,5 @@
     <xacro:include filename="$(find my_robot_arm)/urdf/links_joints.xacro"/>
     <xacro:property name="h1" value=".3"/>
-    <xacro:property name="d2" value=".2"/>
+    <xacro:property name="d2" value=".3"/>
     <xacro:property name="d3" value=".3"/>
     <!-- BASE -->
