Commit message: modif urdf

File: urdf/links_joints.xacro (robot description, xacro)
@@ -1,3 +1,9 @@
 <?xml version="1.0"?>
+<!--
+# Macros para la creación de articulaciones, eslabones de tipo rotacional, prismático y fijo,
+# y para la creación de la pinza del elemento terminal
+#
+# Gabriel Montoiro Varela
+-->
 <robot name="my_robot_arm_macros" xmlns:xacro="http://www.ros.org/wiki/xacro">
     <xacro:macro name="m_joint_r" params="name min max axis_xyz origin_rpy origin_xyz parent child">
@@ -45,50 +51,4 @@
                 <geometry>
 	            <box size="${size}"/>
-                </geometry>
-            </visual>
-        </link>
-    </xacro:macro>
-    <xacro:macro name="gripper_dh" params="name material">
-        <link name="${name}">
-            <visual>
-                <origin rpy="0 0 .78" xyz="0 0 0"/>
-                <material name="${material}"/>
-                <geometry>
-                    <box size="0.01 0.1 0.01"/>
-                </geometry>
-            </visual>
-            <visual>
-                <origin rpy="0 0 .78" xyz="0 0 0"/>
-                <material name="${material}"/>
-                <geometry>
-                    <box size="0.1 0.01 0.01"/>
-                </geometry>
-            </visual>
-            <visual>
-                <origin rpy="0 0 .78" xyz=".0318 -.0318 0.01"/>
-                <material name="${material}"/>
-                <geometry>
-                    <box size="0.01 0.01 0.03"/>
-                </geometry>
-            </visual>
-            <visual>
-                <origin rpy="0 0 .78" xyz="-.0318 .0318 0.01"/>
-                <material name="${material}"/>
-                <geometry>
-                    <box size="0.01 0.01 0.03"/>
-                </geometry>
-            </visual>
-            <visual>
-                <origin rpy="0 0 .78" xyz=".0318 .0318 0.01"/>
-                <material name="${material}"/>
-                <geometry>
-                    <box size="0.01 0.01 0.03"/>
-                </geometry>
-            </visual>
-            <visual>
-                <origin rpy="0 0 .78" xyz="-.0318 -.0318 0.01"/>
-                <material name="${material}"/>
-                <geometry>
-                    <box size="0.01 0.01 0.03"/>
                 </geometry>
             </visual>

File: urdf/my_robot_arm.xacro (robot description, xacro)
@@ -1,5 +1,12 @@
 <?xml version="1.0"?>
+<!--
+# Modelo de brazo robotíco 6DOF 2RP3R (tipo Stanford)
+#
+# Gabriel Montoiro Varela
+-->
 <robot name="my_robot_arm" xmlns:xacro="http://www.ros.org/wiki/xacro">
+    <!-- definición de macros -->
     <xacro:include filename="$(find my_robot_arm)/urdf/links_joints.xacro"/>
+    <!-- dimensiones de los eslabones -->
     <xacro:property name="h1" value=".3"/>
     <xacro:property name="d2" value=".3"/>
